Commit message: update

File: ridgeback/ridgeback_description/urdf/test.urdf (robot description, URDF)
Before this commit: robot ridgeback, 71 links, 70 joints
Joints:
- joint robotiq_coupler_joint: origin xyz=0 0 0.06 rpy=-1.57079632679 0 -3.14159265359 -> xyz=0 0 0.06 rpy=-1.57079632679 0 -3.92699081699
- joint robotiq_hand_joint: origin xyz=0 0 0.004 rpy=0 -1.57079632679 3.14159265359 -> xyz=0 0 0.004 rpy=0 0 3.14159265359
- joint ur_base_link_joint: origin xyz=0.28 0.0 0 rpy=0.0 0.0 -1.5708 -> xyz=0.28 0.0 0 rpy=0.0 0.0 -0.785398163397

Commit message: update mecanum_drive_controller

File: ridgeback/ridgeback_description/urdf/test.urdf (robot description, URDF)
Before this commit: robot ridgeback, 71 links, 70 joints
Links:
- link finger_1_link_0: geometry collision mesh filename=package://robotiq_3f_gripper_visualization/meshes/robotiq-3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; visual mesh filename=package://robotiq_3f_gripper_visualization/meshes/robotiq-3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
- link finger_1_link_1: geometry collision mesh filename=package://robotiq_3f_gripper_visualization/meshes/robotiq-3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; visual mesh filename=package://robotiq_3f_gripper_visualization/meshes/robotiq-3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
- link finger_1_link_2: geometry collision mesh filename=package://robotiq_3f_gripper_visualization/meshes/robotiq-3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; visual mesh filename=package://robotiq_3f_gripper_visualization/meshes/robotiq-3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
- link finger_1_link_3: geometry collision mesh filename=package://robotiq_3f_gripper_visualization/meshes/robotiq-3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; visual mesh filename=package://robotiq_3f_gripper_visualization/meshes/robotiq-3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
- link finger_2_link_0: geometry collision mesh filename=package://robotiq_3f_gripper_visualization/meshes/robotiq-3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; visual mesh filename=package://robotiq_3f_gripper_visualization/meshes/robotiq-3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
- link finger_2_link_1: geometry collision mesh filename=package://robotiq_3f_gripper_visualization/meshes/robotiq-3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; visual mesh filename=package://robotiq_3f_gripper_visualization/meshes/robotiq-3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
- link finger_2_link_2: geometry collision mesh filename=package://robotiq_3f_gripper_visualization/meshes/robotiq-3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; visual mesh filename=package://robotiq_3f_gripper_visualization/meshes/robotiq-3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
- link finger_2_link_3: geometry collision mesh filename=package://robotiq_3f_gripper_visualization/meshes/robotiq-3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; visual mesh filename=package://robotiq_3f_gripper_visualization/meshes/robotiq-3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
- link finger_middle_link_0: geometry collision mesh filename=package://robotiq_3f_gripper_visualization/meshes/robotiq-3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; visual mesh filename=package://robotiq_3f_gripper_visualization/meshes/robotiq-3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
- link finger_middle_link_1: geometry collision mesh filename=package://robotiq_3f_gripper_visualization/meshes/robotiq-3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; visual mesh filename=package://robotiq_3f_gripper_visualization/meshes/robotiq-3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
- link finger_middle_link_2: geometry collision mesh filename=package://robotiq_3f_gripper_visualization/meshes/robotiq-3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; visual mesh filename=package://robotiq_3f_gripper_visualization/meshes/robotiq-3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
- link finger_middle_link_3: geometry collision mesh filename=package://robotiq_3f_gripper_visualization/meshes/robotiq-3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; visual mesh filename=package://robotiq_3f_gripper_visualization/meshes/robotiq-3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
- link palm: geometry collision box size=0.1 0.1 0.1; visual mesh filename=package://robotiq_3f_gripper_visualization/meshes/robotiq-3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
