Commit message: update

File: ridgeback/ridgeback_description/urdf/accessories.urdf.xacro (robot description, xacro)
@@ -12,6 +12,7 @@
   <xacro:include filename="$(find ridgeback_description)/urdf/accessories/sick_s300_mount.urdf.xacro" />
   <xacro:include filename="$(find ridgeback_description)/urdf/accessories/hokuyo_ust-10lx_mount.urdf.xacro" />
+  <xacro:include filename="$(find ur_description)/urdf/ur5.urdf.xacro" />
   <!-- If enabled, generate the front HOKUYO UST-10LX LASER payload. -->
-  <xacro:if value="$(optenv RIDGEBACK_FRONT_HOKUYO_LASER 0)">
+  <xacro:if value="$(optenv RIDGEBACK_FRONT_HOKUYO_LASER 1)">
     <xacro:hokuyo_ust-10lx_mount prefix="front"
                                  topic="front/scan"
@@ -25,5 +26,5 @@
   </xacro:if>
   <!-- If enabled, generate the front SICK LMS111 LASER payload. -->
-  <xacro:if value="$(optenv RIDGEBACK_FRONT_SICK_LASER 0)">
+  <xacro:if value="$(optenv RIDGEBACK_FRONT_SICK_LASER 1)">
     <xacro:sick_lms1xx_mount prefix="front"
                              topic="front/scan"
@@ -39,5 +40,5 @@
        This uses the same mesh as the lms1xx since they are the footprint
        and the simulation parameters can be variable. -->
-  <xacro:if value="$(optenv RIDGEBACK_FRONT_S300_LASER 0)">
+  <xacro:if value="$(optenv RIDGEBACK_FRONT_S300_LASER 1)">
     <xacro:sick_s300_mount prefix="front"
                              topic="front/scan"
@@ -59,3 +60,30 @@
     </xacro:microstrain_imu>
   </xacro:if>
+<!-- Spawn arm -->
+  <xacro:ur5_robot prefix="ur5_arm_" joint_limited="true"/>
+  <!-- Join arm -->
+  <joint name="ur5_arm_base" type="fixed">
+	<parent link="chassis_link" />
+	<child link="ur5_arm_base_link" />
+	<origin xyz="0.28 0.0 0" rpy="0.0 0.0 -1.5708" />
+  </joint>
+  <!-- Gripper -->
+  <link name="gripper_link">
+		<visual>
+			<geometry>
+				<box size="0.09 0.13 0.01" />
+			</geometry>
+			<material name="light_grey"/>
+		</visual>
+		<collision>
+			<geometry>
+				<cylinder length="0.04" radius="0.035"/>
+			</geometry>
+		</collision>
+   </link>
+  <joint name="gripper_joint" type="fixed">
+	  <origin xyz="0.005 0.0 0.0" rpy="0.0 1.571 0.0" />
+	  <parent link="ur5_arm_ee_link" />
+	  <child link="gripper_link" />
+  </joint>
 </robot>

File: ridgeback/ridgeback_description/urdf/ridgeback.urdf.xacro (robot description, xacro)
@@ -21,4 +21,5 @@
   <material name="yellow"><color rgba="0.8 0.8 0.0 1.0" /></material>
   <material name="black"><color rgba="0.15 0.15 0.15 1.0" /></material>
+  <xacro:include filename="$(find ur_description)/urdf/ur5.urdf.xacro" />
   <xacro:macro name="wheel" params="prefix side *joint_pose">
     <link name="${prefix}_${side}_wheel_link">

Commit message: update

File: ridgeback/ridgeback_description/urdf/accessories.urdf.xacro (robot description, xacro)
@@ -12,5 +12,5 @@
   <xacro:include filename="$(find ridgeback_description)/urdf/accessories/sick_s300_mount.urdf.xacro" />
   <xacro:include filename="$(find ridgeback_description)/urdf/accessories/hokuyo_ust-10lx_mount.urdf.xacro" />
-  <xacro:include filename="$(find ur_description)/urdf/ur5.urdf.xacro" />
+  <xacro:include filename="$(find ur_description)/urdf/ur5_robotiq.urdf.xacro" />
   <!-- If enabled, generate the front HOKUYO UST-10LX LASER payload. -->
   <xacro:if value="$(optenv RIDGEBACK_FRONT_HOKUYO_LASER 1)">
@@ -20,5 +20,5 @@
   </xacro:if>
   <!-- If enabled, generate the rear HOKUYO UST-10LX LASER payload. -->
-  <xacro:if value="$(optenv RIDGEBACK_REAR_HOKUYO_LASER 0)">
+  <xacro:if value="$(optenv RIDGEBACK_REAR_HOKUYO_LASER 1)">
     <xacro:hokuyo_ust-10lx_mount prefix="rear"
                                  topic="rear/scan"
@@ -32,5 +32,5 @@
   </xacro:if>
   <!-- If enabled, generate the rear SICK LMS111 LASER payload. -->
-  <xacro:if value="$(optenv RIDGEBACK_REAR_SICK_LASER 0)">
+  <xacro:if value="$(optenv RIDGEBACK_REAR_SICK_LASER 1)">
     <xacro:sick_lms1xx_mount prefix="rear"
                              topic="rear/scan"
@@ -64,5 +64,5 @@
   <!-- Join arm -->
   <joint name="ur5_arm_base" type="fixed">
-	<parent link="chassis_link" />
+	<parent link="mid_mount" />
 	<child link="ur5_arm_base_link" />
 	<origin xyz="0.28 0.0 0" rpy="0.0 0.0 -1.5708" />

File: ridgeback/ridgeback_description/urdf/ridgeback.urdf.xacro (robot description, xacro)
@@ -21,5 +21,5 @@
   <material name="yellow"><color rgba="0.8 0.8 0.0 1.0" /></material>
   <material name="black"><color rgba="0.15 0.15 0.15 1.0" /></material>
-  <xacro:include filename="$(find ur_description)/urdf/ur5.urdf.xacro" />
+  <xacro:include filename="$(find ur_description)/urdf/ur5_robotiq.urdf.xacro" />
   <xacro:macro name="wheel" params="prefix side *joint_pose">
     <link name="${prefix}_${side}_wheel_link">

Commit message: 保持官方版本

File: ridgeback/ridgeback_description/urdf/accessories.urdf.xacro (robot description, xacro)
@@ -1,4 +1,4 @@
 <?xml version="1.0"?>
-<robot xmlns:xacro="http://www.ros.org/wiki/xacro">
+<robot xmlns:xacro="http://ros.org/wiki/xacro">
   <!--
     As you add to this URDF, please be aware that both the robot and
@@ -12,8 +12,6 @@
   <xacro:include filename="$(find ridgeback_description)/urdf/accessories/sick_s300_mount.urdf.xacro" />
   <xacro:include filename="$(find ridgeback_description)/urdf/accessories/hokuyo_ust-10lx_mount.urdf.xacro" />
-  <xacro:include filename="$(find ridgeback_description)/urdf/accessories/microstrain_imu.urdf.xacro" />
-  <xacro:include filename="$(find ur_description)/urdf/ur5_robotiq.urdf.xacro" />
   <!-- If enabled, generate the front HOKUYO UST-10LX LASER payload. -->
-  <xacro:if value="$(optenv RIDGEBACK_FRONT_HOKUYO_LASER 1)">
+  <xacro:if value="$(optenv RIDGEBACK_FRONT_HOKUYO_LASER 0)">
     <xacro:hokuyo_ust-10lx_mount prefix="front"
                                  topic="front/scan"
@@ -61,36 +59,3 @@
     </xacro:microstrain_imu>
   </xacro:if>
-<!-- Spawn arm -->
-<!--
-  <xacro:ur5_robot prefix="ur5_arm_" joint_limited="true"/>
--->
-  <!-- Join arm -->
-  <!--
-  <joint name="ur5_arm_base" type="fixed">
-	<parent link="mid_mount" />
-	<child link="ur5_arm_base_link" />
-	<origin xyz="0.28 0.0 0" rpy="0.0 0.0 -1.5708" />
-  </joint>
--->
-  <!-- Gripper -->
-  <!--
-  <link name="gripper_link">
-		<visual>
-			<geometry>
-				<box size="0.09 0.13 0.01" />
-			</geometry>
-			<material name="light_grey"/>
-		</visual>
-		<collision>
-			<geometry>
-				<cylinder length="0.04" radius="0.035"/>
-			</geometry>
-		</collision>
-   </link>
-  <joint name="gripper_joint" type="fixed">
-	  <origin xyz="0.005 0.0 0.0" rpy="0.0 1.571 0.0" />
-	  <parent link="ur5_arm_ee_link" />
-	  <child link="gripper_link" />
-  </joint>
--->
 </robot>

File: ridgeback/ridgeback_description/urdf/accessories/hokuyo_ust-10lx_mount.urdf.xacro (robot description, xacro)
@@ -1,4 +1,4 @@
 <?xml version="1.0"?>
-<robot xmlns:xacro="http://www.ros.org/wiki/xacro">
+<robot xmlns:xacro="http://ros.org/wiki/xacro">
   <xacro:macro name="hokuyo_ust-10lx_mount" params="prefix topic location">
     <joint name="${prefix}_laser_joint" type="fixed">

File: ridgeback/ridgeback_description/urdf/accessories/microstrain_imu.urdf.xacro (robot description, xacro)
@@ -1,4 +1,4 @@
 <?xml version="1.0"?>
-<robot xmlns:xacro="http://www.ros.org/wiki/xacro">
+<robot xmlns:xacro="http://ros.org/wiki/xacro">
   <xacro:macro name="microstrain_imu" params="prefix mount_link *joint_pose">
   <link name="${prefix}_imu_link" >

File: ridgeback/ridgeback_description/urdf/accessories/sick_lms1xx_mount.urdf.xacro (robot description, xacro)
@@ -24,5 +24,5 @@
 SOFTWARE, EVEN IF ADVISED OF THE POSSIBILITY OF SUCH DAMAGE.
 -->
-<robot xmlns:xacro="http://www.ros.org/wiki/xacro">
+<robot xmlns:xacro="http://ros.org/wiki/xacro">
   <xacro:include filename="$(find lms1xx)/urdf/sick_lms1xx.urdf.xacro" />
   <xacro:macro name="sick_lms1xx_mount" params="prefix topic location">

File: ridgeback/ridgeback_description/urdf/accessories/sick_s300_mount.urdf.xacro (robot description, xacro)
@@ -24,5 +24,5 @@
 SOFTWARE, EVEN IF ADVISED OF THE POSSIBILITY OF SUCH DAMAGE.
 -->
-<robot xmlns:xacro="http://www.ros.org/wiki/xacro">
+<robot xmlns:xacro="http://ros.org/wiki/xacro">
   <xacro:include filename="$(find lms1xx)/urdf/sick_lms1xx.urdf.xacro" />
   <xacro:macro name="sick_s300_mount" params="prefix topic location">

File: ridgeback/ridgeback_description/urdf/test.urdf (robot description, URDF)
Before this commit: robot ridgeback, 71 links, 70 joints
Links:
- removed link base
- removed link ee_link
- removed link finger_1_link_0
- removed link finger_1_link_1
- removed link finger_1_link_2
- removed link finger_1_link_3
- removed link finger_1_link_median_actuating_hinge
- removed link finger_1_link_median_bar
- removed link finger_1_link_median_bar_underactuated
- removed link finger_1_link_paradistal_hinge
- removed link finger_1_link_paramedian_hinge
- removed link finger_1_link_paraproximal_actuating_hinge
- removed link finger_1_link_paraproximal_bar
- removed link finger_1_link_proximal_actuating_bar
- removed link finger_1_link_proximal_actuating_hinge
- removed link finger_2_link_0
- removed link finger_2_link_1
- removed link finger_2_link_2
- removed link finger_2_link_3
- removed link finger_2_link_median_actuating_hinge
- removed link finger_2_link_median_bar
- removed link finger_2_link_median_bar_underactuated
- removed link finger_2_link_paradistal_hinge
- removed link finger_2_link_paramedian_hinge
- removed link finger_2_link_paraproximal_actuating_hinge
- removed link finger_2_link_paraproximal_bar
- removed link finger_2_link_proximal_actuating_bar
- removed link finger_2_link_proximal_actuating_hinge
- removed link finger_middle_link_0
- removed link finger_middle_link_1
- removed link finger_middle_link_2
- removed link finger_middle_link_3
- removed link finger_middle_link_median_actuating_hinge
- removed link finger_middle_link_median_bar
- removed link finger_middle_link_median_bar_underactuated
- removed link finger_middle_link_paradistal_hinge
- removed link finger_middle_link_paramedian_hinge
- removed link finger_middle_link_paraproximal_actuating_hinge
- removed link finger_middle_link_paraproximal_bar
- removed link finger_middle_link_proximal_actuating_bar
- removed link finger_middle_link_proximal_actuating_hinge
- removed link forearm_link
- removed link front_laser
- removed link grasping_frame
- removed link palm
- removed link robotiq_coupler
- removed link shoulder_link
- removed link tool0
- removed link upper_arm_link
- removed link ur_base_link
- removed link wrist_1_link
- removed link wrist_2_link
- removed link wrist_3_link
Joints:
- removed joint base_link-base_fixed_joint
- removed joint ee_fixed_joint
- removed joint elbow_joint
- removed joint finger_1_joint_1
- removed joint finger_1_joint_2
- removed joint finger_1_joint_3
- removed joint finger_1_joint_median_actuating_hinge
- removed joint finger_1_joint_median_actuating_hinge_median_bar
- removed joint finger_1_joint_paradistal_hinge
- removed joint finger_1_joint_paramedian_hinge
- removed joint finger_1_joint_paramedian_hinge_median_bar_underactuated
- removed joint finger_1_joint_paraproximal_actuating_hinge
- removed joint finger_1_joint_paraproximal_bar
- removed joint finger_1_joint_proximal_actuating_bar
- removed joint finger_1_joint_proximal_actuating_hinge
- removed joint finger_2_joint_1
- removed joint finger_2_joint_2
- removed joint finger_2_joint_3
- removed joint finger_2_joint_median_actuating_hinge
- removed joint finger_2_joint_median_actuating_hinge_median_bar
- removed joint finger_2_joint_paradistal_hinge
- removed joint finger_2_joint_paramedian_hinge
- removed joint finger_2_joint_paramedian_hinge_median_bar_underactuated
- removed joint finger_2_joint_paraproximal_actuating_hinge
- removed joint finger_2_joint_paraproximal_bar
- removed joint finger_2_joint_proximal_actuating_bar
- removed joint finger_2_joint_proximal_actuating_hinge
- removed joint finger_middle_joint_1
- removed joint finger_middle_joint_2
- removed joint finger_middle_joint_3
- removed joint finger_middle_joint_median_actuating_hinge
- removed joint finger_middle_joint_median_actuating_hinge_median_bar
- removed joint finger_middle_joint_paradistal_hinge
- removed joint finger_middle_joint_paramedian_hinge
- removed joint finger_middle_joint_paramedian_hinge_median_bar_underactuated
- removed joint finger_middle_joint_paraproximal_actuating_hinge
- removed joint finger_middle_joint_paraproximal_bar
- removed joint finger_middle_joint_proximal_actuating_bar
- removed joint finger_middle_joint_proximal_actuating_hinge
- removed joint front_laser_joint
- removed joint grasping_frame_joint
- removed joint palm_finger_1_joint
- removed joint palm_finger_2_joint
- removed joint palm_finger_middle_joint
- removed joint robotiq_coupler_joint
- removed joint robotiq_hand_joint
- removed joint shoulder_lift_joint
- removed joint shoulder_pan_joint
- removed joint ur_base_link_joint
- removed joint wrist_1_joint
- removed joint wrist_2_joint
- removed joint wrist_3_joint
- removed joint wrist_3_link-tool0_fixed_joint
